File: HallBox.kicad_pcb (KiCad board)
At the start: 2 copper layers, 282.7 x 136.2 mm, 88 parts, among them J1 USB C Connector, J2 JTAG_TC2030, SW1 Boot, U1 XC6206, U2 USBLC6-2SC6, U3 RP2040, U4 W25Q128JVS, Y1 12MHz

Commit message: updated pcb
Routing:
- added copper zone on F.Cu, net GND
Changed lines of the file:
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@@
     )
   )
-  (zone (net 2) (net_name "GND") (layer "B.Cu") (hatch edge 0.508)
+  (zone (net 2) (net_name "GND") (layers "F&B.Cu") (hatch edge 0.508)
     (connect_pads (clearance 0.508))
     (min_thickness 0.254) (filled_areas_thickness no)
